Commit message: feat: MoveIt Setup Assistant - 配置 MoveIt Config 包并验证

File: src/dm_arm_description/urdf/dm_arm_description.urdf (robot description, URDF)
Before this commit: robot dm_arm_description, 12 links, 11 joints
Joints:
- joint gripper_left: limit lower=-0.045 upper=0.0 effort=20 velocity=0.2 -> lower=-0.045 upper=0.0 effort=20.0 velocity=0.2
- joint gripper_right: limit lower=-0.045 upper=0.0 effort=20 velocity=0.2 -> lower=-0.045 upper=0.0 effort=20.0 velocity=0.2
- joint joint1: limit lower=-2.0943951023931953 upper=2.0943951023931953 effort=100 velocity=3 -> lower=-2.0943951023931953 upper=2.0943951023931953 effort=100.0 velocity=3.0
- joint joint2: limit lower=0.0 upper=3.141592653589793 effort=100 velocity=3 -> lower=0.0 upper=3.141592653589793 effort=100.0 velocity=3.0
- joint joint3: limit lower=0.0 upper=4.71238898038469 effort=100 velocity=3 -> lower=0.0 upper=4.71238898038469 effort=100.0 velocity=3.0
- joint joint4: limit lower=-1.5707963267948966 upper=1.5707963267948966 effort=20 velocity=3 -> lower=-1.5707963267948966 upper=1.5707963267948966 effort=20.0 velocity=3.0
- joint joint5: limit lower=-1.5707963267948966 upper=1.5707963267948966 effort=20 velocity=3 -> lower=-1.5707963267948966 upper=1.5707963267948966 effort=20.0 velocity=3.0
- joint joint6: limit lower=-3.141592653589793 upper=3.141592653589793 effort=20 velocity=3 -> lower=-3.141592653589793 upper=3.141592653589793 effort=20.0 velocity=3.0
